Commit message: gripper poses position process

File: src/ros2_robotiq_gripper/robotiq_description/urdf/robotiq_2f_85_gripper.urdf.xacro (robot description, xacro)
@@ -4,9 +4,14 @@
     <xacro:arg name="com_port" default="/dev/ttyUSB0" />
     <xacro:include filename="$(find robotiq_description)/urdf/robotiq_2f_85_macro.urdf.xacro" />
-    <link name="world" />
+    <link name="base_floating">
+        <inertial>
+            <mass value="0.5"/>
+            <inertia ixx="1e-3" ixy="0" ixz="0" iyy="1e-3" iyz="0" izz="1e-3"/>
+        </inertial>
+    </link>
     <xacro:robotiq_gripper
         name="RobotiqGripperHardwareInterface"
         prefix=""
-        parent="world"
+        parent="base_floating"
         use_fake_hardware="$(arg use_fake_hardware)"
         com_port="$(arg com_port)"
